File: 33NJU23/33NJU23.kicad_sch (KiCad schematic)
At the start: 72 parts, among them CN1 HDMI, J1 VGA, J10 Conn_01x02, J11 Conn_01x01, J12 Audio OUT, J13 Audio IN, J14 JOY-1, J15 USB_A, J17 USB_B_Micro, J18 Conn_01x02_Female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

Commit message: create
Parts:
- Q1, Q2: footprint LIBS:SOT-23_PLUS -> LIBS:SOT-23_PLUS2
Changed lines of the file:
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@@
       (effects (font (size 1.27 1.27)) (justify left))
     )
-    (property "Footprint" "LIBS:SOT-23_PLUS" (id 2) (at 165.1 163.195 0)
+    (property "Footprint" "LIBS:SOT-23_PLUS2" (id 2) (at 165.1 163.195 0)
       (effects (font (size 1.27 1.27) italic) (justify left) hide)
     )
@@
       (effects (font (size 1.27 1.27)) (justify left))
     )
-    (property "Footprint" "LIBS:SOT-23_PLUS" (id 2) (at 147.32 170.815 0)
+    (property "Footprint" "LIBS:SOT-23_PLUS2" (id 2) (at 147.32 170.815 0)
       (effects (font (size 1.27 1.27) italic) (justify left) hide)
     )
@@
     )
     (path "/e5ad4f1c-6e58-4293-bc7a-575d8112a533"
-      (reference "Q1") (unit 1) (value "BC850") (footprint "LIBS:SOT-23_PLUS")
+      (reference "Q1") (unit 1) (value "BC850") (footprint "LIBS:SOT-23_PLUS2")
     )
     (path "/3337ae61-4c2b-4233-849f-051dc653cdde"
-      (reference "Q2") (unit 1) (value "BC850") (footprint "LIBS:SOT-23_PLUS")
+      (reference "Q2") (unit 1) (value "BC850") (footprint "LIBS:SOT-23_PLUS2")
     )
     (path "/56d3bec8-62e0-4b75-8a5f-35a1fc1ba854"
