File: 33NJU23/33NJU23.kicad_pcb (KiCad board)
At the start: 2 copper layers, 54 x 85.7 mm, 75 parts, among them CN1 HDMI, J1 VGA, J10 Conn_01x02, J11 Conn_01x01, J12 Audio OUT, J13 Audio IN, J14 JOY-1, J15 USB_A, J17 USB_B_Micro, J18 Conn_01x02_Female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

Commit message: .
Changed lines of the file:
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@@
       (effects (font (size 1 1) (thickness 0.15)))
     )
-    (fp_text user "C5" (at 0 0 180 unlocked) (layer "B.SilkS")
+    (fp_text user "C5" (at 0 0 unlocked) (layer "B.SilkS")
       (effects (font (size 0.8 0.8) (thickness 0.15)) (justify mirror))
     )
@@
     (fp_line (start -1.67 39.16) (end -1.67 39.58) (layer "F.SilkS") (width 0.12))
     (fp_line (start 19.45 1.06) (end 19.45 1.48) (layer "F.SilkS") (width 0.12))
-    (fp_arc (start 19.42 49.32) (mid 19.213487 49.588772) (end 18.89 49.69) (layer "F.SilkS") (width 0.12))
-    (fp_arc (start 18.89 -1.43) (mid 19.213484 -1.328785) (end 19.42 -1.06) (layer "F.SilkS") (width 0.12))
+    (fp_arc (start 19.42 49.32) (mid 19.213496 49.58881) (end 18.89 49.69) (layer "F.SilkS") (width 0.12))
+    (fp_arc (start 18.89 -1.43) (mid 19.213502 -1.328793) (end 19.42 -1.06) (layer "F.SilkS") (width 0.12))
     (fp_arc (start -1.11 49.69) (mid -1.433508 49.588809) (end -1.64 49.32) (layer "F.SilkS") (width 0.12))
     (fp_arc (start -1.64 -1.06) (mid -1.433508 -1.328808) (end -1.11 -1.43) (layer "F.SilkS") (width 0.12))

Commit message: create
Parts:
- Q1, Q2: footprint LIBS:SOT-23_PLUS -> LIBS:SOT-23_PLUS2
- moved Q2 1.53 mm to (66.2, 85.1), turned to 180 degrees
- moved Q1 0.71 mm to (59.4, 83.7)
- moved C9 0.35 mm to (41.3, 56.1)
Routing:
- net /RIGHT_OUT: track 60.3 -> 54.5 mm
- net /LOAD_IN_D: track 37.2 -> 41.9 mm
- net /LEFT_OUT: track 60.5 -> 57.6 mm
- net Net-(D1-Pad1): track 14.7 -> 17.3 mm, vias 0 -> 1
- net Net-(D1-Pad2): track 21.7 -> 24.2 mm
- net /BEEP_OUT: track 55.5 -> 53.1 mm
- net Net-(Q2-Pad1): track 5.65 -> 8.01 mm
- net /PS/2_DATA_3V: track 70.7 -> 69.7 mm
- net /PS/2_CLK_3V: track 77.4 -> 76.7 mm

Commit message: logo
Parts:
- added G***: LOGO, LOGO, F.Cu at (60.3, 68.7)
Routing:
- net GND: track 554.6 -> 574.3 mm, vias 16 -> 18
- net /GP_4: track 27.8 -> 30.6 mm

Commit message: .
Parts:
- moved G*** 0.13 mm to (60.3, 68.6)
Routing:
- net GND: track 574.3 -> 590.3 mm, vias 18 -> 19
- net /R*: track 23.2 -> 11.6 mm
- net /L: track 38.4 -> 34.0 mm
- net /R: track 35.6 -> 38.8 mm
- net /GP_15: track 51.3 -> 49.8 mm
- net Net-(C3-Pad2): track 8.56 -> 7.14 mm
- net /+3V3: track 180.8 -> 181.6 mm
- net /PS/2_DATA_3V: track 69.7 -> 70.4 mm
- net /RIGHT_OUT: track 54.5 -> 54.0 mm
- net /LOAD_IN: track 29.6 -> 29.1 mm

Commit message: reload
Changed lines of the file:
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@@
     (fp_line (start -1.67 39.16) (end -1.67 39.58) (layer "F.SilkS") (width 0.12))
     (fp_line (start 19.45 1.06) (end 19.45 1.48) (layer "F.SilkS") (width 0.12))
-    (fp_arc (start 19.42 49.32) (mid 19.213497 49.588778) (end 18.89 49.69) (layer "F.SilkS") (width 0.12))
-    (fp_arc (start 18.89 -1.43) (mid 19.213502 -1.328793) (end 19.42 -1.06) (layer "F.SilkS") (width 0.12))
+    (fp_arc (start 19.42 49.32) (mid 19.213487 49.588772) (end 18.89 49.69) (layer "F.SilkS") (width 0.12))
+    (fp_arc (start 18.89 -1.43) (mid 19.213484 -1.328785) (end 19.42 -1.06) (layer "F.SilkS") (width 0.12))
     (fp_arc (start -1.11 49.69) (mid -1.433508 49.588809) (end -1.64 49.32) (layer "F.SilkS") (width 0.12))
     (fp_arc (start -1.64 -1.06) (mid -1.433508 -1.328808) (end -1.11 -1.43) (layer "F.SilkS") (width 0.12))
@@
   )
   (dimension (type aligned) (layer "F.Fab")
+    (pts (xy 78.105 97.79) (xy 78.105 110.49))
+    (height -17.78)
+    (gr_text "12,7000 мм" (at 94.735 104.14 90) (layer "F.Fab")
+      (effects (font (size 1 1) (thickness 0.15)))
+    )
+    (format (units 3) (units_format 1) (precision 4))
+    (style (thickness 0.1) (arrow_length 1.27) (text_position_mode 0) (extension_height 0.58642) (extension_offset 0.5) keep_text_aligned)
+  )
+  (dimension (type aligned) (layer "F.Fab")
     (pts (xy 83.82 118.745) (xy 74.676 118.745))
     (height 3.048)
@@
   )
   (dimension (type aligned) (layer "F.Fab")
+    (pts (xy 33.02 110.363) (xy 56.373448 110.363))
+    (height 7.366)
+    (gr_text "23,3534 мм" (at 44.696724 116.579) (layer "F.Fab")
+      (effects (font (size 1 1) (thickness 0.15)))
+    )
+    (format (units 3) (units_format 1) (precision 4))
+    (style (thickness 0.1) (arrow_length 1.27) (text_position_mode 0) (extension_height 0.58642) (extension_offset 0.5) keep_text_aligned)
+  )
+  (dimension (type aligned) (layer "F.Fab")
+    (pts (xy 24.892 89.408) (xy 24.892 67.945))
+    (height 1.905)
+    (gr_text "21,4630 мм" (at 25.647 78.6765 90) (layer "F.Fab")
+      (effects (font (size 1 1) (thickness 0.15)))
+    )
+    (format (units 3) (units_format 1) (precision 4))
+    (style (thickness 0.1) (arrow_length 1.27) (text_position_mode 0) (extension_height 0.58642) (extension_offset 0.5) keep_text_aligned)
+  )
+  (dimension (type aligned) (layer "F.Fab")
     (pts (xy 62.84 28.026) (xy 83.82 28.026))
     (height -6.944)
@@
       (effects (font (size 1 1) (thickness 0.15)))
     )
+    (format (units 3) (units_format 1) (precision 4))
+    (style (thickness 0.1) (arrow_length 1.27) (text_position_mode 0) (extension_height 0.58642) (extension_offset 0.5) keep_text_aligned)
+  )
+  (dimension (type aligned) (layer "F.Fab")
+    (pts (xy 36.195 67.945) (xy 36.195 92.456))
+    (height 14.478)
+    (gr_text "24,5110 мм" (at 20.567 80.2005 90) (layer "F.Fab")
+      (effects (font (size 1 1) (thickness 0.15)))
+    )
+    (format (units 3) (units_format 1) (precision 4))
+    (style (thickness 0.1) (arrow_length 1.27) (text_position_mode 0) (extension_height 0.58642) (extension_offset 0.5) keep_text_aligned)
+  )
+  (dimension (type aligned) (layer "F.Fab")
+    (pts (xy 24.13 102.616) (xy 24.13 92.456))
+    (height 3.175)
+    (gr_text "10,1600 мм" (at 26.155 97.536 90) (layer "F.Fab")
+      (effects (font (size 1 1) (thickness 0.15)))
+    )
