File: 33EJU23/33EJU23.kicad_pcb (KiCad board)
At the start: 2 copper layers, 54 x 85.7 mm, 107 parts, among them CN1 HDMI, J1 VGA, J10 Conn_01x02, J11 Conn_01x03, J12 VIDEO, J13 Conn_02x05_Odd_Even, J2 EXT, J3 JOY-1, J4 USB_A, J5 USB_A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

Commit message: .
Parts:
- added R33: 1к5, Resistor_SMD:R_0805_2012Metric_Pad1.20x1.40mm_HandSolder, B.Cu at (62.7, 63.9)
- added R34: 1k5, Resistor_SMD:R_0805_2012Metric_Pad1.20x1.40mm_HandSolder, B.Cu at (60.6, 64.6)
- added R35: 1k5, Resistor_SMD:R_0805_2012Metric_Pad1.20x1.40mm_HandSolder, B.Cu at (58.4, 64.7)
- R20, R23, R26: value 330 -> 390
- R21, R24, R27: value 1k -> 820
Routing:
- net /GP_13: track 0.45 -> 20.1 mm, vias 0 -> 1
- net /G_IN0: track 11.0 -> 16.8 mm
- net GND: track 183.4 -> 189.1 mm
- net /D+: track 42.8 -> 46.3 mm
- net /B_IN0: track 5.83 -> 8.39 mm
- net /SYNC: track 62.2 -> 63.3 mm

Commit message: create
Routing:
- net /D-: track 41.8 -> 45.3 mm
Changed lines of the file:
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@@
     (property "Sheetfile" "33EJU23.kicad_sch")
     (property "Sheetname" "")
-    (attr smd)
+    (attr through_hole)
     (fp_text reference "J3" (at 7.7724 0.0283 90) (layer "F.SilkS")
       (effects (font (size 1 1) (thickness 0.15)))
@@
   (segment (start 46.228 38.862) (end 46.285 38.805) (width 0.3) (layer "B.Cu") (net 59))
   (segment (start 62.5896 35.127) (end 62.5896 36.195) (width 0.3) (layer "F.Cu") (net 61))
-  (segment (start 63.5896 39.4496) (end 64.145 40.005) (width 0.2) (layer "F.Cu") (net 61))
+  (segment (start 63.5896 35.127) (end 63.5896 35.9784) (width 0.3) (layer "F.Cu") (net 61))
+  (segment (start 63.5896 35.9784) (end 63.5896 39.4496) (width 0.3) (layer "F.Cu") (net 61))
   (segment (start 62.865 36.195) (end 62.5896 36.195) (width 0.3) (layer "F.Cu") (net 61))
-  (segment (start 63.5896 35.127) (end 63.5896 36.152) (width 0.3) (layer "F.Cu") (net 61))
   (segment (start 63.5896 36.152) (end 63.5896 39.4496) (width 0.2) (layer "F.Cu") (net 61))
   (segment (start 63.5896 33.894893) (end 63.5896 35.127) (width 0.3) (layer "F.Cu") (net 61))
   (segment (start 63.5396 36.202) (end 62.872 36.202) (width 0.3) (layer "F.Cu") (net 61))
+  (segment (start 63.5896 39.4496) (end 64.145 40.005) (width 0.3) (layer "F.Cu") (net 61))
   (segment (start 63.487945 33.793238) (end 63.5896 33.894893) (width 0.3) (layer "F.Cu") (net 61))
   (segment (start 63.5896 36.152) (end 63.5396 36.202) (width 0.3) (layer "F.Cu") (net 61))
   (segment (start 63.487945 32.534506) (end 63.487945 33.793238) (width 0.3) (layer "F.Cu") (net 61))
+  (segment (start 63.5896 35.9784) (end 63.5896 36.152) (width 0.3) (layer "F.Cu") (net 61))
   (segment (start 62.872 36.202) (end 62.865 36.195) (width 0.3) (layer "F.Cu") (net 61))
   (segment (start 62.354207 67.945) (end 67.691 62.608207) (width 0.4) (layer "B.Cu") (net 61))

Commit message: logo
Parts:
- removed the C_5V at (64.8, 106.4)
- added G***: LOGO, LOGO, F.Cu at (35.5, 92.4)
- G***: moved to B.Cu
- moved G*** 34.0 mm to (64.8, 108.7), turned to 180 degrees
Routing:
- net GND: track 189.1 -> 222.1 mm, vias 18 -> 19
- net /ANT: track 39.0 -> 50.0 mm
- net /+5V: track 281.6 -> 276.4 mm
- net /FSC: track 24.9 -> 24.2 mm
Other:
- board text added: "12M"
- board text added: "16M"
- board text added: "4.43M"

Commit message: .
Parts:
- removed the G*** at (64.8, 108.7)
- removed the G*** at (47.0, 108.5)
- added C_3V: 10u, Capacitor_SMD:C_0805_2012Metric_Pad1.18x1.45mm_HandSolder, B.Cu at (75.3, 89.0)
- added i2c: , LIBS:Crystal_SMD_0603-4Pin_6.0x3.5mm, B.Cu at (64.8, 107.0)
- G***: moved to F.Cu
- moved G*** 17.8 mm to (47.0, 108.8), turned to 0 degrees
- moved C_5V 1.45 mm to (75.9, 107.7)
Routing:
- net GND: track 222.1 -> 261.6 mm
- net /+3V3: track 64.8 -> 89.2 mm
- net /GP_14: track 26.2 -> 50.5 mm
- net /GP_15: track 31.6 -> 48.0 mm, vias 2 -> 3
Other:
- outline, holes or cut-outs redrawn
- board text added: "Notch Up"
