File: 33EJU23/33EJU23.kicad_sch (KiCad schematic)
At the start: 87 parts, among them CN1 HDMI, J1 VGA, J10 Conn_01x02, J11 Conn_01x03, J12 VIDEO, J13 Conn_02x05_Odd_Even, J2 EXT, J3 JOY-1, J4 USB_A, J5 USB_A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

Commit message: .
Parts:
- added R33: 1к5, Resistor_SMD:R_0805_2012Metric_Pad1.20x1.40mm_HandSolder, symbol Device:R
- added R34, R35: 1k5, Resistor_SMD:R_0805_2012Metric_Pad1.20x1.40mm_HandSolder, symbol Device:R
- R20, R23, R26: value 330 -> 390
- R21, R24, R27: value 1k -> 820
Connections:
- net B_IN0: now also R35.1
- net GP_13: now also R33.2, R34.2, R35.2
- net G_IN0: now also R34.1
- net R_IN0: now also R33.1
Other:
- moved on the sheet: C1, C3, C4, C5, J4, J5, J6, J7, JP4, JP5, R10, R11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

Commit message: reload
Parts:
- C17: value 0.1u -> 0.1u||1k*
- C21: value 10n -> 1n
- R18: value 100 -> 200-1k*
- R19: value 100 -> 1R
- R20, R23, R26: value 390 -> 1k
- R21, R24, R27: value 820 -> 2k
- R22, R25, R28: value 100* -> 200*
- R29: value 100* -> 1k
- R32: value 100* -> 10-30*
- R33: value 1к5 -> -
- R34, R35: value 1k5 -> -
Other:
- note added: "R33-R35 не запаивать!!!"
- note added: "запаять 1-2 или 2-3"
- note added: "запаять либо R30 либо R31,R32"
